Commit message: Robot aux dimensions reelles Adept Rev B (datasheet officiel)
- URDF : 1.051 x 0.494 x 0.425 m (au lieu de 0.45 x 0.35 x 0.15)
- Roues : rayon 0.203 m (16" pneumatique) au lieu de 0.085
- Masses : 60 kg chassis + 4x8 kg roues (77 kg reels)
- wheel_separation 0.563 m ESTIMÉ (largeur totale - largeur pneu),
  a mesurer au lab pour raffinage
- Impact : plugin DiffDrive Gazebo, driver ROS, simulateur protocole
- Valide en sim : robot proportionné, cul-de-sac 3x3 confortable,
  conduite fluide dans galeries 3 m
- Fondation nav2 correcte avant N5

File: src/seekur_driver/urdf/seekur_jr_simple.urdf.xacro (robot description, xacro)
@@ -4,15 +4,18 @@
     <xacro:arg name="robot_color" default="Grey"/>
     <xacro:property name="robot_color" value="$(arg robot_color)"/>
-    <!-- Propriétés SeekurJR -->
-    <xacro:property name="base_length" value="0.45" />
-    <xacro:property name="base_width" value="0.35" />
-    <xacro:property name="base_height" value="0.15" />
-    <xacro:property name="wheel_radius" value="0.085" />
-    <xacro:property name="wheel_length" value="0.05" />
-    <xacro:property name="wheel_separation" value="0.33" />
-    <!-- Masses SeekurJR -->
-    <xacro:property name="base_mass" value="25.0" />
-    <xacro:property name="wheel_mass" value="2.0" />
-    <xacro:property name="caster_mass" value="0.5" />
+    <!-- =======================================================
+         Proprietes SeekurJR - Datasheet officiel Adept Rev B
+         (SeekurJr-Datasheet-RevB.pdf, 2011, Adept MobileRobots)
+         ======================================================= -->
+    <xacro:property name="base_length" value="1.051" />      <!-- 1051 mm datasheet -->
+    <xacro:property name="base_width" value="0.494" />       <!-- 494 mm chassis hors roues -->
+    <xacro:property name="base_height" value="0.425" />      <!-- 425 mm hauteur chassis -->
+    <xacro:property name="wheel_radius" value="0.203" />     <!-- 16" pneumatique = 406 mm diam -->
+    <xacro:property name="wheel_length" value="0.10" />      <!-- largeur pneu approx 10 cm -->
+    <xacro:property name="wheel_separation" value="0.563" /> <!-- ESTIME : largeur_totale (663) - largeur_pneu (100). A MESURER AU LAB. -->
+    <!-- Masses (datasheet : robot complet 77 kg) -->
+    <xacro:property name="base_mass" value="60.0" />         <!-- chassis + electronique -->
+    <xacro:property name="wheel_mass" value="8.0" />         <!-- 16" pneumatique ~8 kg piece -->
+    <xacro:property name="caster_mass" value="0.5" />        <!-- non present sur vrai SeekurJR, garde pour stabilite Gazebo -->
     <!-- Couleurs -->
     <material name="blue"><color rgba="0 0 0.8 1" /></material>
@@ -172,6 +175,6 @@
             <left_joint>base_left_wheel_joint</left_joint>
             <right_joint>base_right_wheel_joint</right_joint>
-            <wheel_separation>0.33</wheel_separation>
-            <wheel_radius>0.085</wheel_radius>
+            <wheel_separation>0.563</wheel_separation>      <!-- MAJ Rev B -->
+            <wheel_radius>0.203</wheel_radius>              <!-- MAJ Rev B -->
             <topic>cmd_vel</topic>
             <odom_topic>odom</odom_topic>

Commit message: Fidelite dimensionnelle : wheel_separation constructeur + LiDAR avant
- wheel_separation : 0.563 (estime) -> 0.68 m (URDF officiel Adept
  amr-ros-config, plugin skid-steer). Valeur cinematique effective
  qui inclut le glissement des roues, pas juste l'entraxe geometrique
  (0.312 x 2). Impact : urdf xacro, driver, simulateur.
- LiDAR deplace du toit vers l'avant en saillie, mi-hauteur chassis :
  x=0.55, z=0.10 relatif base_link (~0.30 m du sol) - reflete le
  montage reel du robot UQAT (photo 2026-08). A affiner au mm pres
  au lab si besoin.
- Carte SLAM conservee : murs verticaux pleins => coupe 2D independante
  de la hauteur du plan de scan. TF gere le reste.
- Valide : navigation autonome nav2 reste operationnelle avec les
  nouvelles dimensions et position LiDAR (goals proche et lointain,
  evitement obstacles dynamiques).

File: src/seekur_driver/urdf/seekur_jr_simple.urdf.xacro (robot description, xacro)
@@ -13,5 +13,5 @@
     <xacro:property name="wheel_radius" value="0.203" />     <!-- 16" pneumatique = 406 mm diam -->
     <xacro:property name="wheel_length" value="0.10" />      <!-- largeur pneu approx 10 cm -->
-    <xacro:property name="wheel_separation" value="0.563" /> <!-- ESTIME : largeur_totale (663) - largeur_pneu (100). A MESURER AU LAB. -->
+    <xacro:property name="wheel_separation" value="0.68" /> <!-- ESTIME : largeur_totale (663) - largeur_pneu (100). A MESURER AU LAB. -->
     <!-- Masses (datasheet : robot complet 77 kg) -->
     <xacro:property name="base_mass" value="60.0" />         <!-- chassis + electronique -->
@@ -169,5 +169,9 @@
         <parent link="base_link" />
         <child link="laser_frame" />
-        <origin xyz="0.12 0 ${base_height + 0.035}" rpy="0 0 0" />
+        <!-- LiDAR monte a l'AVANT en saillie, centre optique a mi-hauteur
+            chassis (photo robot UQAT 2026-08). x=0.55 (devant le chassis),
+            z=0.10 relatif a base_link (=0.30 m du sol). A affiner par
+            mesure physique precise au lab. -->
+        <origin xyz="0.55 0 0.10" rpy="0 0 0" />
     </joint>
     <gazebo>
@@ -175,5 +179,5 @@
             <left_joint>base_left_wheel_joint</left_joint>
             <right_joint>base_right_wheel_joint</right_joint>
-            <wheel_separation>0.563</wheel_separation>      <!-- MAJ Rev B -->
+            <wheel_separation>0.68</wheel_separation>      <!-- MAJ Rev B -->
             <wheel_radius>0.203</wheel_radius>              <!-- MAJ Rev B -->
             <topic>cmd_vel</topic>

Commit message: P1 complet: fusion inertielle EKF (IMU + odometrie roues)
P1a - IMU simule :
- Link imu_link + joint au centre chassis (mi-hauteur)
- Capteur type imu 100Hz, bruit MPU9250, gz-sim-imu-system
- Bridge /imu/data public (GZ_TO_ROS)
- Valide : gravite 9.81 sur Z, gyro reactif en rotation

P1b - Fusion EKF (robot_localization) :
- ekf.yaml : EKF 2D, vx roues + vyaw gyro (cle anti-derive skid-steer)
- sim_ekf.launch.py : chaine + EKF, driver publish_tf:=false
- sim.launch.py : argument publish_tf (defaut true, non regressif)
- EKF proprietaire unique de odom->base_footprint

RESULTAT VALIDE (test rotation) :
- Sans fusion : derive angulaire progressive Gazebo vs RViz (roues
  skid-steer glissent en rotation)
- Avec fusion : angle synchronise Gazebo/RViz, derive corrigee par gyro
- Limite connue : patinage translation pure non corrige (IMU seul)

Piege corrige : YAML rcl strict type mixte int/float -> 0 devient 0.0

Base posee pour recalage absolu futur (RFID/BLE/AprilTag) et RTAB-Map.

File: src/seekur_driver/urdf/seekur_jr_simple.urdf.xacro (robot description, xacro)
@@ -143,4 +143,18 @@
                                o_xyz="0 0 0" o_rpy="0 0 0" />
     </link>
+    <!-- IMU Link : centre du robot (bonne pratique fusion : proche du
+         centre de rotation, minimise les accelerations parasites en rotation).
+         Petit box symbolique, inertie negligeable mais non nulle (exigence Gazebo). -->
+    <link name="imu_link">
+        <visual>
+            <geometry>
+                <box size="0.03 0.03 0.02" />
+            </geometry>
+            <origin xyz="0 0 0" rpy="0 0 0" />
+            <material name="red" />
+        </visual>
+        <xacro:box_inertia m="0.05" x="0.03" y="0.03" z="0.02"
+                          o_xyz="0 0 0" o_rpy="0 0 0" />
+    </link>
     <!-- Joints -->
     <joint name="base_joint" type="fixed">
@@ -160,4 +174,13 @@
         <origin xyz="${-base_length / 4.0} ${(base_width + wheel_length) / 2.0} 0" rpy="0 0 0" />
         <axis xyz="0 1 0" />
+    </joint>
+    <!-- IMU monte au CENTRE geometrique du chassis, a mi-hauteur.
+         Centre de rotation du robot -> minimise les artefacts d'acceleration
+         centripete quand le robot tourne. base_link est au sol via base_joint,
+         donc z = base_height/2 place l'IMU a mi-hauteur du chassis. -->
+    <joint name="imu_joint" type="fixed">
+        <parent link="base_link" />
+        <child link="imu_link" />
+        <origin xyz="0 0 ${base_height / 2.0}" rpy="0 0 0" />
     </joint>
     <joint name="base_caster_wheel_joint" type="fixed">
@@ -210,4 +233,11 @@
         <plugin filename="gz-sim-sensors-system" name="gz::sim::systems::Sensors">
             <render_engine>ogre2</render_engine>
+        </plugin>
+    </gazebo>
+    <!-- Systeme IMU : indispensable pour que le capteur type "imu" produise
+         des donnees. Distinct de gz-sim-sensors-system (qui gere lidar/camera).
+         Sans ce systeme, le <sensor type="imu"> reste muet. -->
+    <gazebo>
+        <plugin filename="gz-sim-imu-system" name="gz::sim::systems::Imu">
         </plugin>
     </gazebo>
@@ -241,4 +271,31 @@
         </sensor>
     </gazebo>
+    <!-- Capteur IMU : gyro 3 axes + accelerometre 3 axes.
+         Bruit calibre type MPU9250 (valeurs generiques realistes).
+         NOTE : l'IMU interne du vrai SeekurJR (paquets 0x9A) n'a jamais
+         ete confirme fonctionnel (dump reel ne montrait que des SIP 0x32).
+         Plan B au lab : IMU externe MPU9250 (package imu_serial_reader
+         du NaviBot). L'EKF consomme /imu/data quelle que soit la source. -->
+    <gazebo reference="imu_link">
+        <sensor name="imu_sensor" type="imu">
+            <pose>0 0 0 0 0 0</pose>
+            <topic>imu/data</topic>
+            <gz_frame_id>imu_link</gz_frame_id>
+            <update_rate>100</update_rate>
+            <always_on>1</always_on>
+            <imu>
+                <angular_velocity>
+                    <x><noise type="gaussian"><mean>0.0</mean><stddev>2e-4</stddev></noise></x>
+                    <y><noise type="gaussian"><mean>0.0</mean><stddev>2e-4</stddev></noise></y>
+                    <z><noise type="gaussian"><mean>0.0</mean><stddev>2e-4</stddev></noise></z>
+                </angular_velocity>
+                <linear_acceleration>
+                    <x><noise type="gaussian"><mean>0.0</mean><stddev>1.7e-2</stddev></noise></x>
+                    <y><noise type="gaussian"><mean>0.0</mean><stddev>1.7e-2</stddev></noise></y>
+                    <z><noise type="gaussian"><mean>0.0</mean><stddev>1.7e-2</stddev></noise></z>
+                </linear_acceleration>
+            </imu>
+        </sensor>
+    </gazebo>
     <!-- Propriétés Gazebo -->
     <gazebo reference="base_link">

Commit message: P2: camera RealSense D455 simulee (RGB + depth + pointcloud)
Modele :
- Link camera_link + camera_optical_frame (convention RealSense/ROS,
  RPY -pi/2,0,-pi/2) monte sur mat a xyz=0.3 0 0.6 relatif base_link
  Position ESTIMEE, a mesurer au lab.
- Capteur Gazebo rgbd_camera, 848x480 @ 30 Hz, FOV 90 deg,
  clip depth 0.6-6.0 m (spec D455)

Bridges renommes vers les conventions realsense2_camera :
  /camera/image        -> /camera/color/image_raw
  /camera/depth_image  -> /camera/depth/image_rect_raw
  /camera/points       -> /camera/depth/color/points
  /camera/camera_info  -> /camera/color/camera_info
Le passage sim -> vrai robot ne demandera aucun changement des
configs YOLO/RTAB-Map en aval (meme philosophie que /odom public).

PREREQUIS ENVIRONNEMENT : CycloneDDS obligatoire.
  export RMW_IMPLEMENTATION=rmw_cyclonedds_cpp
  paquet ros-jazzy-rmw-cyclonedds-cpp
Avec FastDDS (defaut Jazzy) les topics camera s'effondrent a 6-13 Hz
avec des blocages de ~1 s : echec de reconstitution des messages
fragmentes sur loopback. Avec Cyclone : 26.9 Hz recus pour 26.9 Hz
produits, ecart-type 0.008 s, zero perte.
Causes ecartees pendant le diagnostic (documentees dans le xacro) :
GPU, Gazebo, RViz, resolution, buffers UDP noyau.

Correctifs environnement au passage (hors depot) :
- Driver NVIDIA repare : headers kernel 7.0.0-30 manquants empechaient
  l'assemblage des modules .ko. Gazebo lance via PRIME offload
  (alias ros2nv dans ~/.bashrc).
- colcon build SANS --symlink-install pour seekur_driver : le symlink
  invalidait les metadonnees Python (PackageNotFoundError au lancement
  des noeuds).

File: src/seekur_driver/urdf/seekur_jr_simple.urdf.xacro (robot description, xacro)
@@ -157,4 +157,34 @@
                           o_xyz="0 0 0" o_rpy="0 0 0" />
     </link>
+    <!-- ================================================================
+         Camera RealSense D455 : montee sur mat au-dessus du chassis.
+         Convention frames RealSense/ROS :
+           - camera_link          : convention robot (X vers l'avant)
+           - camera_optical_frame : convention optique (Z vers la scene,
+                                    X droite, Y bas) - c'est ce frame_id
+                                    que RTAB-Map, YOLO ROS, RViz attendent
+                                    dans le header des images.
+         Le sensor Gazebo est declare sur camera_link (regarde vers +X du
+         link, donc vers l'avant du robot). Le gz_frame_id force le frame
+         optique dans les messages ROS -> memes conventions que le vrai
+         driver realsense2_camera.
+         ================================================================ -->
+    <link name="camera_link">
+        <visual>
+            <!-- D455 : 124 x 26 x 29 mm approximatif (bandeau caviar) -->
+            <geometry>
+                <box size="0.026 0.124 0.029" />
+            </geometry>
+            <origin xyz="0 0 0" rpy="0 0 0" />
+            <material name="black" />
+        </visual>
+        <xacro:box_inertia m="0.1" x="0.026" y="0.124" z="0.029"
+                          o_xyz="0 0 0" o_rpy="0 0 0" />
+    </link>
+    <!-- Frame optique : rotation ROS -> optique. Convention standard :
+         RPY = (-pi/2, 0, -pi/2) fait que Z_optique aligne avec X_link,
+         X_optique aligne avec -Y_link, Y_optique aligne avec -Z_link.
+         C'est LA convention utilisee par tous les drivers de camera ROS. -->
+    <link name="camera_optical_frame" />
     <!-- Joints -->
     <joint name="base_joint" type="fixed">
@@ -197,4 +227,21 @@
             mesure physique precise au lab. -->
         <origin xyz="0.55 0 0.10" rpy="0 0 0" />
+    </joint>
+    <!-- Camera sur mat : legerement devant le centre du chassis, ~60 cm
+         au-dessus de base_link (~80 cm du sol total). Position ESTIMEE,
+         a mesurer au lab. Le mat lui-meme n'est pas modelise visuellement
+         (detail cosmetique) - on modelise juste la position de la camera
+         qui compte pour la simulation. -->
+    <joint name="camera_joint" type="fixed">
+        <parent link="base_link" />
+        <child link="camera_link" />
+        <origin xyz="0.3 0 0.6" rpy="0 0 0" />
+    </joint>
+    <!-- Joint optique : rotation qui aligne le repere optique standard
+         (Z vers la scene) avec le repere robot (X vers la scene). -->
+    <joint name="camera_optical_joint" type="fixed">
+        <parent link="camera_link" />
+        <child link="camera_optical_frame" />
+        <origin xyz="0 0 0" rpy="${-pi/2} 0 ${-pi/2}" />
     </joint>
     <gazebo>
@@ -298,4 +345,64 @@
         </sensor>
     </gazebo>
+    <!-- Capteur RGBD Intel RealSense D455 (simule).
+         Un seul capteur rgbd_camera Gazebo Harmonic produit :
+           - image RGB     (color)
+           - image depth   (aligned sur RGB)
+           - point cloud   (depth reprojete + couleur)
+           - camera_info
+         Spec D455 reproduites :
+           - FOV RGB   90 deg horizontal (Intel : 90x65)
+           - FOV depth 87 deg horizontal (Intel : 87x58) - approx via un seul
+             FOV rgbd (compromis, Gazebo n'expose qu'un HFOV commun)
+           - Resolution 848x480 @ 30 Hz (native RealSense, adapte YOLO/RTAB)
+             REQUIERT CycloneDDS - voir commentaire sur update_rate
+           - Portee depth clip 0.6 - 6.0 m (spec D455)
+         gz_frame_id=camera_optical_frame -> les messages sortent avec le
+         frame optique dans le header (RTAB-Map/YOLO/RViz OK). Le sensor
+         est physiquement attache a camera_link (X pointe vers la scene),
+         mais l'annotation ROS pointe vers camera_optical_frame. -->
+    <gazebo reference="camera_link">
+        <sensor name="camera_d455" type="rgbd_camera">
+            <pose>0 0 0 0 0 0</pose>
+            <topic>camera</topic>
+            <gz_frame_id>camera_optical_frame</gz_frame_id>
+            <!-- PREREQUIS CRITIQUE : CycloneDDS (RMW_IMPLEMENTATION=
+                 rmw_cyclonedds_cpp). Avec FastDDS (defaut Jazzy), les
+                 topics image/depth/pointcloud s'effondrent a 6-13 Hz avec
+                 des blocages de ~1 s, quelle que soit la resolution.
+                 Diagnostic 2026-08, causes ECARTEES une par une :
+                   - GPU        : RTX 4060 a 32% d'utilisation, large marge
+                   - Gazebo     : produisait bien 14.4 Hz (mesure gz topic)
+                   - RViz       : aucun effet une fois retire
+                   - Resolution : reduire de 3x a EMPIRE le debit
+                   - Buffers UDP noyau (rmem/wmem max) : aucun effet
+                 Cause reelle : fragmentation DDS des gros messages sur
+                 loopback. Une image 848x480 RGB depasse largement le seuil
+                 de fragmentation ; FastDDS echoue a reconstituer, Cyclone
+                 y arrive sans peine.
+                 Apres bascule CycloneDDS : 14.4 Hz recus pour 14.4 Hz
+                 produits, ecart-type 0.006 s. Zero perte. -->
+            <update_rate>30</update_rate>
+            <always_on>1</always_on>
+            <camera>
+                <horizontal_fov>1.5708</horizontal_fov> <!-- 90 deg = pi/2 -->
+                <!-- 848x480 : resolution native RealSense D455. -->
+                <image>
+                    <width>848</width>
+                    <height>480</height>
+                    <format>R8G8B8</format>
+                </image>
+                <clip>
+                    <near>0.6</near>
+                    <far>6.0</far>
+                </clip>
+                <noise>
+                    <type>gaussian</type>
+                    <mean>0.0</mean>
+                    <stddev>0.007</stddev>
+                </noise>
+            </camera>
+        </sensor>
+    </gazebo>
     <!-- Propriétés Gazebo -->
     <gazebo reference="base_link">
@@ -316,3 +423,6 @@
         <material>Gazebo/Blue</material>
     </gazebo>
+    <gazebo reference="camera_link">
+        <material>Gazebo/Black</material>
+    </gazebo>
 </robot>
