Commit message: test/tripode : chassis v10.0 (2 roues AR + roulette AV) + capteurs 40169fd, LiDAR horizontal
mine_gallery, RTAB-Map 0.23.7, ~98 m : 9 fermetures globales, 3 de proximite
(v10.1 meme jour : 1 et 0). Le basculement du chassis 4 appuis (+/-3.3 deg,
mesure IMU sim) etait la cause de la chute des fermetures.

File: src/seekur_driver/urdf/seekur_jr_simple.urdf.xacro (robot description, xacro)
@@ -17,6 +17,5 @@
                           494 = hauteur totale du robot
                           425 = empattement (axe avant - axe arriere)
-                                (utilise UNIQUEMENT pour placer les 4 roues
-                                visuelles ; la physique reste a 2 roues + 2 roulettes)
+                                (non utilise ici : modele a 2 roues + roulette)
          ATTENTION - deux erreurs corrigees par rapport aux versions
          precedentes de ce fichier :
@@ -37,12 +36,4 @@
     <xacro:property name="wheel_length" value="0.165" />     <!-- [DS] 6.50" de section = 165 mm -->
     <xacro:property name="wheel_separation" value="0.663" /> <!-- [DS] 663 mm ; confirme [LAB] a 3 mm pres -->
-    <xacro:property name="lidar_pitch_deg" value="5" />      <!-- [SIM] inclinaison LiDAR vers le haut -->
-    <xacro:property name="wheelbase" value="0.425" />        <!-- [DS] 425 mm ; visuels seulement (voir roues visuelles) -->
-    <!-- Maillages visuels (modele Blender, exporte en OBJ dans le repere
-         base_link : axe des roues a z = 0, avant vers +X, fond du chassis
-         a -chassis_drop, haut a chassis_top). file:// + $(find) est resolu
-         a la fois par RViz2 et par Gazebo Harmonic (package:// ne l'est
-         pas toujours cote Gazebo). -->
-    <xacro:property name="mesh_dir" value="file://$(find seekur_driver)/description/meshes" />
     <!-- Mat de camera. Le top du chassis est a (base_height - chassis_drop)
          dans base_link, soit 0.291 m ; la camera se deduit de la hauteur du
@@ -59,10 +50,5 @@
     <xacro:property name="base_mass" value="60.0" />         <!-- chassis + electronique -->
     <xacro:property name="wheel_mass" value="8.0" />         <!-- 16" pneumatique ~8 kg piece -->
-    <xacro:property name="caster_mass" value="0.5" />        <!-- par roulette ; non present sur vrai SeekurJR, garde pour stabilite Gazebo -->
-    <xacro:property name="caster_radius" value="${wheel_radius / 2.0}" />
-    <xacro:property name="caster_x" value="${base_length / 3.0}" />  <!-- roulettes a +/- 0.35 m -->
-    <xacro:property name="caster_gap" value="0.02" />       <!-- 2 cm au-dessus du sol (bosses de la mine) : les 2 roues motrices
-                                                                  gardent toujours le contact (4 appuis en
-                                                                  losange = hyperstatique sinon) -->
+    <xacro:property name="caster_mass" value="0.5" />        <!-- non present sur vrai SeekurJR, garde pour stabilite Gazebo -->
     <!-- Couleurs -->
     <material name="blue"><color rgba="0 0 0.8 1" /></material>
@@ -109,12 +95,10 @@
          le decalage -chassis_drop applique aux trois origines ci-dessous. -->
     <link name="base_link">
-        <!-- Visuel : maillage deja exprime dans le repere base_link, donc
-             origine nulle. PAS de <material> : il remplacerait les couleurs
-             du .mtl par une teinte unie (RViz2 et Gazebo). -->
-        <visual>
-            <geometry>
-                <mesh filename="${mesh_dir}/seekurjr_chassis.obj" />
-            </geometry>
-            <origin xyz="0 0 0" rpy="0 0 0" />
+        <visual>
+            <geometry>
+                <box size="${base_length} ${base_width} ${base_height}" />
+            </geometry>
+            <origin xyz="0 0 ${base_height / 2.0 - chassis_drop}" rpy="0 0 0" />
+            <material name="robot_material"/>
         </visual>
         <collision>
@@ -127,8 +111,12 @@
                           o_xyz="0 0 ${base_height / 2.0 - chassis_drop}" o_rpy="0 0 0" />
     </link>
-    <!-- Roue motrice right : PHYSIQUE SEULEMENT (collision + inertie).
-         Pas de visuel : ce sont les 4 roues visuelles, aux positions
-         reelles, qui s'affichent (voir plus bas). -->
     <link name="right_wheel_link">
+        <visual>
+            <geometry>
+                <cylinder radius="${wheel_radius}" length="${wheel_length}" />
+            </geometry>
+            <origin xyz="0 0 0" rpy="${pi / 2.0} 0 0" />
+            <material name="black" />
+        </visual>
         <collision>
             <geometry>
@@ -140,8 +128,12 @@
                                o_xyz="0 0 0" o_rpy="${pi / 2.0} 0 0" />
     </link>
-    <!-- Roue motrice left : PHYSIQUE SEULEMENT (collision + inertie).
-         Pas de visuel : ce sont les 4 roues visuelles, aux positions
-         reelles, qui s'affichent (voir plus bas). -->
     <link name="left_wheel_link">
+        <visual>
+            <geometry>
+                <cylinder radius="${wheel_radius}" length="${wheel_length}" />
+            </geometry>
+            <origin xyz="0 0 0" rpy="${pi / 2.0} 0 0" />
+            <material name="black" />
+        </visual>
         <collision>
             <geometry>
@@ -153,81 +145,21 @@
                                o_xyz="0 0 0" o_rpy="${pi / 2.0} 0 0" />
     </link>
-    <!-- Roulettes AVANT et ARRIERE : PHYSIQUE SEULEMENT (absentes du vrai
-         SeekurJR). Elles equilibrent le modele diff-drive dont les roues
-         motrices sont au centre (x = 0). Spheres quasi sans frottement,
-         surelevees de caster_gap : le robot bascule d'au plus ~3.3 deg (2 cm)
-         sur l'une d'elles, les roues motrices ne decollent jamais.
-         Pas de visuel (masquees par le chassis maille). -->
-    <xacro:macro name="caster" params="name x">
-        <link name="${name}_caster_link">
-            <collision>
-                <geometry>
-                    <sphere radius="${caster_radius}" />
-                </geometry>
-                <origin xyz="0 0 0" rpy="0 0 0" />
-            </collision>
-            <xacro:sphere_inertia m="${caster_mass}" r="${caster_radius}"
-                                 o_xyz="0 0 0" o_rpy="0 0 0" />
-        </link>
-        <joint name="base_${name}_caster_joint" type="fixed">
-            <parent link="base_link" />
-            <child link="${name}_caster_link" />
-            <!-- bas de la sphere a caster_gap du sol (sol a z = -wheel_radius) -->
-            <origin xyz="${x} 0 ${-wheel_radius + caster_radius + caster_gap}" rpy="0 0 0" />
-        </joint>
-        <gazebo reference="${name}_caster_link">
-            <mu1 value="0.001" />
-            <mu2 value="0.001" />
-        </gazebo>
-    </xacro:macro>
-    <xacro:caster name="front" x="${caster_x}" />
-    <xacro:caster name="rear"  x="${-caster_x}" />
-    <!-- ================================================================
-         Roues VISUELLES : les 4 roues du vrai SeekurJR, a leurs positions
-         reelles (x = +/- wheelbase/2, y = +/- wheel_separation/2).
-         - Aucune collision : la physique reste portee par les 2 roues
-           motrices centrales + les 2 roulettes.
-         - Joint continuous avec <mimic> sur la roue motrice du meme cote :
-           robot_state_publisher calcule leur angle a partir de
-           /joint_states, donc elles tournent dans RViz des que les 2 joints
-           moteurs sont publies (Gazebo en sim ; driver option B en reel).
-         - Inertie minuscule mais non nulle : Gazebo ignore un link sans
-           inertie relie par un joint mobile.
-         - Gazebo (DART) ne supporte pas les contraintes mimic : il affiche
-           une fois "[Err] ... does not support mimic constraints" au
-           demarrage. ATTENDU ET SANS EFFET : dans Gazebo, ces roues sont
-           entrainees par le plugin DiffDrive (joints ajoutes a sa liste) ;
-           dans RViz, par robot_state_publisher via le mimic.
-         - yaw : le maillage de roue n'est pas symetrique (moyeu/axe d'un
-           cote). pi a GAUCHE, 0 a DROITE : l'axe du moyeu pointe vers
-           l'interieur, cote chassis (valide visuellement dans RViz).
-         ================================================================ -->
-    <xacro:macro name="visual_wheel" params="name x y yaw mimic_joint">
-        <link name="${name}_wheel_visual_link">
-            <visual>
-                <geometry>
-                    <mesh filename="${mesh_dir}/seekurjr_wheel.obj" />
-                </geometry>
-                <origin xyz="0 0 0" rpy="0 0 ${yaw}" />
-            </visual>
-            <xacro:cylinder_inertia m="0.01" r="${wheel_radius}" l="${wheel_length}"
-                                   o_xyz="0 0 0" o_rpy="${pi / 2.0} 0 0" />
-        </link>
-        <joint name="${name}_wheel_visual_joint" type="continuous">
-            <parent link="base_link" />
-            <child link="${name}_wheel_visual_link" />
-            <origin xyz="${x} ${y} 0" rpy="0 0 0" />
-            <axis xyz="0 1 0" />
-            <mimic joint="${mimic_joint}" multiplier="1.0" offset="0.0" />
-        </joint>
-    </xacro:macro>
-    <xacro:visual_wheel name="front_left"  x="${wheelbase / 2.0}"  y="${wheel_separation / 2.0}"
-                        yaw="${pi}" mimic_joint="base_left_wheel_joint" />
-    <xacro:visual_wheel name="rear_left"   x="${-wheelbase / 2.0}" y="${wheel_separation / 2.0}"
-                        yaw="${pi}" mimic_joint="base_left_wheel_joint" />
-    <xacro:visual_wheel name="front_right" x="${wheelbase / 2.0}"  y="${-wheel_separation / 2.0}"
-                        yaw="0"     mimic_joint="base_right_wheel_joint" />
-    <xacro:visual_wheel name="rear_right"  x="${-wheelbase / 2.0}" y="${-wheel_separation / 2.0}"
-                        yaw="0"     mimic_joint="base_right_wheel_joint" />
+    <link name="caster_wheel_link">
+        <visual>
+            <geometry>
+                <sphere radius="${wheel_radius / 2.0}" />
+            </geometry>
+            <origin xyz="0 0 0" rpy="0 0 0" />
+            <material name="black" />
+        </visual>
+        <collision>
+            <geometry>
+                <sphere radius="${wheel_radius / 2.0}" />
+            </geometry>
+            <origin xyz="0 0 0" rpy="0 0 0" />
+        </collision>
+        <xacro:sphere_inertia m="${caster_mass}" r="${wheel_radius / 2.0}"
+                             o_xyz="0 0 0" o_rpy="0 0 0" />
+    </link>
     <!-- LiDAR Link -->
     <link name="laser_frame">
@@ -237,5 +169,5 @@
             </geometry>
             <origin xyz="0 0 0" rpy="0 0 0" />
-            <material name="grey" />
+            <material name="blue" />
         </visual>
         <collision>
@@ -318,20 +250,22 @@
              depuis base_width + wheel_length : le chassis a un gap de
              degagement avec le pneu, les deux grandeurs sont independantes.
-         X : 0. Le vrai robot a 4 roues en skid-steer et pivote au milieu
-             de son empattement (x = 0). Ce modele le represente par un
-             diff-drive EQUIVALENT : 2 roues motrices au centre + roulettes
-             avant/arriere. Meme centre de rotation que le vrai robot, sans
-             les artefacts du skid-steer sous Gazebo (glissement lateral,
-             odometrie de cap faussee, reglage de frottement).
-         HISTORIQUE : jusqu'au 2026-09-24, roues a x = -base_length/4
-         (-0.263) + 1 roulette avant -> pivot decale de 26 cm (ancienne
-         "LIMITE CONNUE"). Les jalons v6 a v9 ont ete valides avec cette
-         geometrie ; a re-valider avec la nouvelle.
-         Les 4 roues VISIBLES sont des links separes (voir plus haut),
-         aux positions reelles, animes par mimic. -->
+         X : -base_length/4. Le vrai robot a 4 roues en skid-steer ; ce
+             modele en a 2 + une roulette avant, donc l'empattement reel
+             (425 mm [DS]) ne s'applique pas ici et n'est pas modelise.
+         LIMITE CONNUE - centre de rotation.
+         Le vrai SeekurJR pivote au milieu de son empattement (x = 0).
+         Ce modele pivote autour de l'axe de ses deux roues (x = -0.263),
+         donc en rotation pure il decrit un arc de 26 cm de rayon au lieu
+         de tourner sur place. Biais systematique, borne, connu.
+         Correction possible le jour ou une rotation reelle est disponible
+         pour comparaison : roues a x = 0 + une seconde roulette a
+         l'arriere pour l'equilibre. Non fait pour l'instant : ce modele
+         est stable dans Gazebo et a servi de base aux jalons v6 a v9,
+         toucher a l'equilibre introduirait un risque non borne pour
+         corriger une erreur qui l'est. -->
     <joint name="base_right_wheel_joint" type="continuous">
         <parent link="base_link" />
         <child link="right_wheel_link" />
-        <origin xyz="0 ${-wheel_separation / 2.0} 0" rpy="0 0 0" />
+        <origin xyz="${-base_length / 4.0} ${-wheel_separation / 2.0} 0" rpy="0 0 0" />
         <axis xyz="0 1 0" />
     </joint>
@@ -339,5 +273,5 @@
         <parent link="base_link" />
         <child link="left_wheel_link" />
-        <origin xyz="0 ${wheel_separation / 2.0} 0" rpy="0 0 0" />
+        <origin xyz="${-base_length / 4.0} ${wheel_separation / 2.0} 0" rpy="0 0 0" />
         <axis xyz="0 1 0" />
     </joint>
@@ -354,4 +288,9 @@
         <child link="imu_link" />
         <origin xyz="0 0 ${-chassis_drop}" rpy="0 0 0" />
+    </joint>
+    <joint name="base_caster_wheel_joint" type="fixed">
+        <parent link="base_link" />
+        <child link="caster_wheel_link" />
+        <origin xyz="${base_length / 3.0} 0 ${-wheel_radius / 2.0}" rpy="0 0 0" />
     </joint>
     <!-- LiDAR SICK, monte en saillie a l'AVANT sur support en equerre.
@@ -370,12 +309,5 @@
         <parent link="base_link" />
         <child link="laser_frame" />
-        <!-- Incline de lidar_pitch_deg vers le HAUT (tangage negatif :
-             en ROS, +pitch fait plonger l'axe X). Evite que le faisceau
-             touche le sol : basculement sur les roulettes (~3.3 deg avec
-             caster_gap 2 cm), bosses et pentes de la mine. Hauteur du
-             faisceau : 0.39 + d*tan(5 deg) -> 0.65 m a 3 m, 2.1 m a 20 m.
-             [SIM] Le support reel doit recevoir la meme inclinaison
-             (cale) ; valeur a remplacer par l'angle mesure. -->
-        <origin xyz="0.535 0 0.187" rpy="0 ${-radians(lidar_pitch_deg)} 0" />
+        <origin xyz="0.535 0 0.187" rpy="0 0 0" />
     </joint>
     <!-- Mat : pose sur le top du chassis, monte de camera_mast_height.
@@ -407,16 +339,6 @@
     <gazebo>
         <plugin filename="libgz-sim-diff-drive-system.so" name="gz::sim::systems::DiffDrive">
-            <!-- Roues motrices physiques : TOUJOURS EN PREMIER. L'odometrie
-                 du plugin est calculee sur le premier joint de chaque cote. -->
             <left_joint>base_left_wheel_joint</left_joint>
             <right_joint>base_right_wheel_joint</right_joint>
-            <!-- Roues VISUELLES (sans collision) : pilotees a la meme vitesse
-                 uniquement pour qu'elles tournent dans la fenetre Gazebo, ou
-                 le mimic n'est pas supporte. Aucun effet physique (pas de
-                 contact, inertie 10 g). RViz, lui, les anime via le mimic. -->
-            <left_joint>front_left_wheel_visual_joint</left_joint>
-            <left_joint>rear_left_wheel_visual_joint</left_joint>
-            <right_joint>front_right_wheel_visual_joint</right_joint>
-            <right_joint>rear_right_wheel_visual_joint</right_joint>
             <!-- Doivent rester coherents avec les proprietes xacro en tete
                  de fichier. Gazebo ne lit pas les ${} ici, d'ou la
@@ -587,8 +509,20 @@
     </gazebo>
     <!-- Propriétés Gazebo -->
-    <!-- base_link et roues : plus de <material> Gazebo, les couleurs
-         viennent des .mtl des maillages. -->
+    <gazebo reference="base_link">
+       <material>Gazebo/Grey</material>
+    </gazebo>
+    <gazebo reference="right_wheel_link">
+        <material>Gazebo/Black</material>
+    </gazebo>
+    <gazebo reference="left_wheel_link">
+        <material>Gazebo/Black</material>
+    </gazebo>
+    <gazebo reference="caster_wheel_link">
+        <material>Gazebo/Black</material>
+        <mu1 value="0.001" />
+        <mu2 value="0.001" />
+    </gazebo>
     <gazebo reference="laser_frame">
-        <material>Gazebo/Grey</material>
+        <material>Gazebo/Blue</material>
     </gazebo>
     <gazebo reference="camera_mast_link">
