Commit message: test/tripode : maillage SeekurJR (db41bde) + traction AVANT (roues x=+L/4, roulette x=-L/3), LiDAR horizontal
mine_polycam : franchit mieux les bosses (roues motrices qui attaquent l'obstacle).

File: src/seekur_driver/urdf/seekur_jr_simple.urdf.xacro (robot description, xacro)
@@ -17,5 +17,6 @@
                           494 = hauteur totale du robot
                           425 = empattement (axe avant - axe arriere)
-                                (non utilise ici : modele a 2 roues + roulette)
+                                (utilise UNIQUEMENT pour placer les 4 roues
+                                visuelles ; la physique reste a 2 roues + roulette)
          ATTENTION - deux erreurs corrigees par rapport aux versions
          precedentes de ce fichier :
@@ -36,4 +37,11 @@
     <xacro:property name="wheel_length" value="0.165" />     <!-- [DS] 6.50" de section = 165 mm -->
     <xacro:property name="wheel_separation" value="0.663" /> <!-- [DS] 663 mm ; confirme [LAB] a 3 mm pres -->
+    <xacro:property name="wheelbase" value="0.425" />        <!-- [DS] 425 mm ; visuels seulement (voir roues visuelles) -->
+    <!-- Maillages visuels (modele Blender, exporte en OBJ dans le repere
+         base_link : axe des roues a z = 0, avant vers +X, fond du chassis
+         a -chassis_drop, haut a chassis_top). file:// + $(find) est resolu
+         a la fois par RViz2 et par Gazebo Harmonic (package:// ne l'est
+         pas toujours cote Gazebo). -->
+    <xacro:property name="mesh_dir" value="file://$(find seekur_driver)/description/meshes" />
     <!-- Mat de camera. Le top du chassis est a (base_height - chassis_drop)
          dans base_link, soit 0.291 m ; la camera se deduit de la hauteur du
@@ -95,10 +103,12 @@
          le decalage -chassis_drop applique aux trois origines ci-dessous. -->
     <link name="base_link">
+        <!-- Visuel : maillage deja exprime dans le repere base_link, donc
+             origine nulle. PAS de <material> : il remplacerait les couleurs
+             du .mtl par une teinte unie (RViz2 et Gazebo). -->
         <visual>
             <geometry>
-                <box size="${base_length} ${base_width} ${base_height}" />
-            </geometry>
-            <origin xyz="0 0 ${base_height / 2.0 - chassis_drop}" rpy="0 0 0" />
-            <material name="robot_material"/>
+                <mesh filename="${mesh_dir}/seekurjr_chassis.obj" />
+            </geometry>
+            <origin xyz="0 0 0" rpy="0 0 0" />
         </visual>
         <collision>
@@ -111,12 +121,8 @@
                           o_xyz="0 0 ${base_height / 2.0 - chassis_drop}" o_rpy="0 0 0" />
     </link>
+    <!-- Roue motrice right : PHYSIQUE SEULEMENT (collision + inertie).
+         Pas de visuel : ce sont les 4 roues visuelles, aux positions
+         reelles, qui s'affichent (voir plus bas). -->
     <link name="right_wheel_link">
-        <visual>
-            <geometry>
-                <cylinder radius="${wheel_radius}" length="${wheel_length}" />
-            </geometry>
-            <origin xyz="0 0 0" rpy="${pi / 2.0} 0 0" />
-            <material name="black" />
-        </visual>
         <collision>
             <geometry>
@@ -128,12 +134,8 @@
                                o_xyz="0 0 0" o_rpy="${pi / 2.0} 0 0" />
     </link>
+    <!-- Roue motrice left : PHYSIQUE SEULEMENT (collision + inertie).
+         Pas de visuel : ce sont les 4 roues visuelles, aux positions
+         reelles, qui s'affichent (voir plus bas). -->
     <link name="left_wheel_link">
-        <visual>
-            <geometry>
-                <cylinder radius="${wheel_radius}" length="${wheel_length}" />
-            </geometry>
-            <origin xyz="0 0 0" rpy="${pi / 2.0} 0 0" />
-            <material name="black" />
-        </visual>
         <collision>
             <geometry>
@@ -145,12 +147,8 @@
                                o_xyz="0 0 0" o_rpy="${pi / 2.0} 0 0" />
     </link>
+    <!-- Roulette : PHYSIQUE SEULEMENT (absente du vrai SeekurJR, gardee
+         pour l'equilibre Gazebo du modele a 2 roues). Pas de visuel : elle
+         apparaissait sous le chassis maille. -->
     <link name="caster_wheel_link">
-        <visual>
-            <geometry>
-                <sphere radius="${wheel_radius / 2.0}" />
-            </geometry>
-            <origin xyz="0 0 0" rpy="0 0 0" />
-            <material name="black" />
-        </visual>
         <collision>
             <geometry>
@@ -162,4 +160,51 @@
                              o_xyz="0 0 0" o_rpy="0 0 0" />
     </link>
+    <!-- ================================================================
+         Roues VISUELLES : les 4 roues du vrai SeekurJR, a leurs positions
+         reelles (x = +/- wheelbase/2, y = +/- wheel_separation/2).
+         - Aucune collision : la physique reste portee par les 2 roues
+           motrices + la roulette (jalons v6 a v9 inchanges).
+         - Joint continuous avec <mimic> sur la roue motrice du meme cote :
+           robot_state_publisher calcule leur angle a partir de
+           /joint_states, donc elles tournent dans RViz des que les 2 joints
+           moteurs sont publies (Gazebo en sim ; driver option B en reel).
+         - Inertie minuscule mais non nulle : Gazebo ignore un link sans
+           inertie relie par un joint mobile.
+         - Gazebo (DART) ne supporte pas les contraintes mimic : il affiche
+           une fois "[Err] ... does not support mimic constraints" au
+           demarrage. ATTENDU ET SANS EFFET : dans Gazebo, ces roues sont
+           entrainees par le plugin DiffDrive (joints ajoutes a sa liste) ;
+           dans RViz, par robot_state_publisher via le mimic.
+         - yaw : le maillage de roue n'est pas symetrique (moyeu/axe d'un
+           cote). pi a GAUCHE, 0 a DROITE : l'axe du moyeu pointe vers
+           l'interieur, cote chassis (valide visuellement dans RViz).
+         ================================================================ -->
+    <xacro:macro name="visual_wheel" params="name x y yaw mimic_joint">
+        <link name="${name}_wheel_visual_link">
+            <visual>
+                <geometry>
+                    <mesh filename="${mesh_dir}/seekurjr_wheel.obj" />
+                </geometry>
+                <origin xyz="0 0 0" rpy="0 0 ${yaw}" />
+            </visual>
+            <xacro:cylinder_inertia m="0.01" r="${wheel_radius}" l="${wheel_length}"
+                                   o_xyz="0 0 0" o_rpy="${pi / 2.0} 0 0" />
+        </link>
+        <joint name="${name}_wheel_visual_joint" type="continuous">
+            <parent link="base_link" />
+            <child link="${name}_wheel_visual_link" />
+            <origin xyz="${x} ${y} 0" rpy="0 0 0" />
+            <axis xyz="0 1 0" />
+            <mimic joint="${mimic_joint}" multiplier="1.0" offset="0.0" />
+        </joint>
+    </xacro:macro>
+    <xacro:visual_wheel name="front_left"  x="${wheelbase / 2.0}"  y="${wheel_separation / 2.0}"
+                        yaw="${pi}" mimic_joint="base_left_wheel_joint" />
+    <xacro:visual_wheel name="rear_left"   x="${-wheelbase / 2.0}" y="${wheel_separation / 2.0}"
+                        yaw="${pi}" mimic_joint="base_left_wheel_joint" />
+    <xacro:visual_wheel name="front_right" x="${wheelbase / 2.0}"  y="${-wheel_separation / 2.0}"
+                        yaw="0"     mimic_joint="base_right_wheel_joint" />
+    <xacro:visual_wheel name="rear_right"  x="${-wheelbase / 2.0}" y="${-wheel_separation / 2.0}"
+                        yaw="0"     mimic_joint="base_right_wheel_joint" />
     <!-- LiDAR Link -->
     <link name="laser_frame">
@@ -169,5 +214,5 @@
             </geometry>
             <origin xyz="0 0 0" rpy="0 0 0" />
-            <material name="blue" />
+            <material name="grey" />
         </visual>
         <collision>
@@ -267,5 +312,5 @@
         <parent link="base_link" />
         <child link="right_wheel_link" />
-        <origin xyz="${-base_length / 4.0} ${-wheel_separation / 2.0} 0" rpy="0 0 0" />
+        <origin xyz="${base_length / 4.0} ${-wheel_separation / 2.0} 0" rpy="0 0 0" />
         <axis xyz="0 1 0" />
     </joint>
@@ -273,5 +318,5 @@
         <parent link="base_link" />
         <child link="left_wheel_link" />
-        <origin xyz="${-base_length / 4.0} ${wheel_separation / 2.0} 0" rpy="0 0 0" />
+        <origin xyz="${base_length / 4.0} ${wheel_separation / 2.0} 0" rpy="0 0 0" />
         <axis xyz="0 1 0" />
     </joint>
@@ -292,5 +337,5 @@
         <parent link="base_link" />
         <child link="caster_wheel_link" />
-        <origin xyz="${base_length / 3.0} 0 ${-wheel_radius / 2.0}" rpy="0 0 0" />
+        <origin xyz="${-base_length / 3.0} 0 ${-wheel_radius / 2.0}" rpy="0 0 0" />
     </joint>
     <!-- LiDAR SICK, monte en saillie a l'AVANT sur support en equerre.
@@ -339,6 +384,16 @@
     <gazebo>
         <plugin filename="libgz-sim-diff-drive-system.so" name="gz::sim::systems::DiffDrive">
+            <!-- Roues motrices physiques : TOUJOURS EN PREMIER. L'odometrie
+                 du plugin est calculee sur le premier joint de chaque cote. -->
             <left_joint>base_left_wheel_joint</left_joint>
             <right_joint>base_right_wheel_joint</right_joint>
+            <!-- Roues VISUELLES (sans collision) : pilotees a la meme vitesse
+                 uniquement pour qu'elles tournent dans la fenetre Gazebo, ou
+                 le mimic n'est pas supporte. Aucun effet physique (pas de
+                 contact, inertie 10 g). RViz, lui, les anime via le mimic. -->
+            <left_joint>front_left_wheel_visual_joint</left_joint>
+            <left_joint>rear_left_wheel_visual_joint</left_joint>
+            <right_joint>front_right_wheel_visual_joint</right_joint>
+            <right_joint>rear_right_wheel_visual_joint</right_joint>
             <!-- Doivent rester coherents avec les proprietes xacro en tete
                  de fichier. Gazebo ne lit pas les ${} ici, d'ou la
@@ -509,13 +564,6 @@
     </gazebo>
     <!-- Propriétés Gazebo -->
-    <gazebo reference="base_link">
-       <material>Gazebo/Grey</material>
-    </gazebo>
-    <gazebo reference="right_wheel_link">
-        <material>Gazebo/Black</material>
-    </gazebo>
-    <gazebo reference="left_wheel_link">
-        <material>Gazebo/Black</material>
-    </gazebo>
+    <!-- base_link et roues : plus de <material> Gazebo, les couleurs
+         viennent des .mtl des maillages. -->
     <gazebo reference="caster_wheel_link">
         <material>Gazebo/Black</material>
@@ -524,5 +572,5 @@
     </gazebo>
     <gazebo reference="laser_frame">
-        <material>Gazebo/Blue</material>
+        <material>Gazebo/Grey</material>
     </gazebo>
     <gazebo reference="camera_mast_link">

Commit message: test/tripode : LiDAR incline de 5 deg vers le haut [SIM]
Sur mine_polycam, l'avant se releve puis replonge sur les bosses ; un LiDAR
horizontal balayait le sol. 5 deg regle le cas courant ; sur une grosse bosse
le scan touche encore parfois le sol (piste : filtrage au sol dans la grille
RTAB-Map). Inclinaison a mesurer sur le vrai robot.

File: src/seekur_driver/urdf/seekur_jr_simple.urdf.xacro (robot description, xacro)
@@ -351,8 +351,9 @@
              biaise les distances mur gauche / mur droit).
              A MESURER : distance centre du boitier <-> axe longitudinal. -->
+    <xacro:property name="lidar_pitch_deg" value="5" />      <!-- [SIM] inclinaison LiDAR vers le haut : evite le sol quand l avant replonge apres une bosse (a mesurer au lab) -->
     <joint name="laser_joint" type="fixed">
         <parent link="base_link" />
         <child link="laser_frame" />
-        <origin xyz="0.535 0 0.187" rpy="0 0 0" />
+        <origin xyz="0.535 0 0.187" rpy="0 ${-radians(lidar_pitch_deg)} 0" />
     </joint>
     <!-- Mat : pose sur le top du chassis, monte de camera_mast_height.

Commit message: Camera renommee camera_front (topics, TF, URDF, bridge, RViz) ; profondeur publiee en aligned_depth_to_color
Nommage par position pour accueillir d'autres cameras (camera_rear, thermal_front).
Topics et profondeur alignes sur le vrai noeud RealSense : un seul reglage
RTAB-Map/YOLO pour la sim et le reel. Valide en sim : topics, 29 Hz, TF,
RTAB-Map, YOLO (person 0.91 a 29.7 Hz).

File: src/seekur_driver/urdf/seekur_jr_simple.urdf.xacro (robot description, xacro)
@@ -246,10 +246,10 @@
          Camera RealSense D455 : montee sur mat au-dessus du chassis.
          Convention frames RealSense/ROS :
-           - camera_link          : convention robot (X vers l'avant)
-           - camera_optical_frame : convention optique (Z vers la scene,
+           - camera_front_link          : convention robot (X vers l'avant)
+           - camera_front_optical_frame : convention optique (Z vers la scene,
                                     X droite, Y bas) - c'est ce frame_id
                                     que RTAB-Map, YOLO ROS, RViz attendent
                                     dans le header des images.
-         Le sensor Gazebo est declare sur camera_link (regarde vers +X du
+         Le sensor Gazebo est declare sur camera_front_link (regarde vers +X du
          link, donc vers l'avant du robot). Le gz_frame_id force le frame
          optique dans les messages ROS -> memes conventions que le vrai
@@ -260,6 +260,6 @@
          flotte en l'air dans RViz et Gazebo), mais il rend le modele
          lisible d'un coup d'oeil. Visual + inertie seulement, pas de
-         collision : meme convention que camera_link et imu_link. -->
-    <link name="camera_mast_link">
+         collision : meme convention que camera_front_link et imu_link. -->
+    <link name="camera_front_mast_link">
         <visual>
             <geometry>
@@ -272,5 +272,5 @@
                                o_xyz="0 0 0" o_rpy="0 0 0" />
     </link>
-    <link name="camera_link">
+    <link name="camera_front_link">
         <visual>
             <!-- D455 : 124 x 26 x 29 mm approximatif (bandeau caviar) -->
@@ -288,5 +288,5 @@
          X_optique aligne avec -Y_link, Y_optique aligne avec -Z_link.
          C'est LA convention utilisee par tous les drivers de camera ROS. -->
-    <link name="camera_optical_frame" />
+    <link name="camera_front_optical_frame" />
     <!-- Joints -->
     <joint name="base_joint" type="fixed">
@@ -369,7 +369,7 @@
     <!-- Mat : pose sur le top du chassis, monte de camera_mast_height.
          Son origine est au milieu du cylindre, d'ou le /2. -->
-    <joint name="camera_mast_joint" type="fixed">
-        <parent link="base_link" />
-        <child link="camera_mast_link" />
+    <joint name="camera_front_mast_joint" type="fixed">
+        <parent link="base_link" />
+        <child link="camera_front_mast_link" />
         <origin xyz="${camera_x} 0 ${chassis_top + camera_mast_height / 2.0}" rpy="0 0 0" />
     </joint>
@@ -381,14 +381,14 @@
                 soit 0.614 m du sol
          y : suppose centree. A confirmer d'un coup d'oeil depuis le dessus. -->
-    <joint name="camera_joint" type="fixed">
-        <parent link="base_link" />
-        <child link="camera_link" />
+    <joint name="camera_front_joint" type="fixed">
+        <parent link="base_link" />
+        <child link="camera_front_link" />
         <origin xyz="${camera_x} 0 ${chassis_top + camera_mast_height}" rpy="0 0 0" />
     </joint>
     <!-- Joint optique : rotation qui aligne le repere optique standard
          (Z vers la scene) avec le repere robot (X vers la scene). -->
-    <joint name="camera_optical_joint" type="fixed">
-        <parent link="camera_link" />
-        <child link="camera_optical_frame" />
+    <joint name="camera_front_optical_joint" type="fixed">
+        <parent link="camera_front_link" />
+        <child link="camera_front_optical_frame" />
         <origin xyz="0 0 0" rpy="${-pi/2} 0 ${-pi/2}" />
     </joint>
@@ -519,13 +519,13 @@
              REQUIERT CycloneDDS - voir commentaire sur update_rate
            - Portee depth clip 0.6 - 6.0 m (spec D455)
-         gz_frame_id=camera_optical_frame -> les messages sortent avec le
+         gz_frame_id=camera_front_optical_frame -> les messages sortent avec le
          frame optique dans le header (RTAB-Map/YOLO/RViz OK). Le sensor
-         est physiquement attache a camera_link (X pointe vers la scene),
-         mais l'annotation ROS pointe vers camera_optical_frame. -->
-    <gazebo reference="camera_link">
+         est physiquement attache a camera_front_link (X pointe vers la scene),
+         mais l'annotation ROS pointe vers camera_front_optical_frame. -->
+    <gazebo reference="camera_front_link">
         <sensor name="camera_d455" type="rgbd_camera">
             <pose>0 0 0 0 0 0</pose>
-            <topic>camera</topic>
-            <gz_frame_id>camera_optical_frame</gz_frame_id>
+            <topic>camera_front</topic>
+            <gz_frame_id>camera_front_optical_frame</gz_frame_id>
             <!-- PREREQUIS CRITIQUE : CycloneDDS (RMW_IMPLEMENTATION=
                  rmw_cyclonedds_cpp). Avec FastDDS (defaut Jazzy), les
@@ -585,8 +585,8 @@
         <material>Gazebo/Grey</material>
     </gazebo>
-    <gazebo reference="camera_mast_link">
+    <gazebo reference="camera_front_mast_link">
         <material>Gazebo/Grey</material>
     </gazebo>
-    <gazebo reference="camera_link">
+    <gazebo reference="camera_front_link">
         <material>Gazebo/Black</material>
     </gazebo>

Commit message: Xacro : inclinaison LiDAR et maillages en arguments (sim par defaut, reel via real.launch.py)
lidar_pitch_deg : 5 [SIM] par defaut, 6.5 [LAB] pour le reel.
mesh_uri : file:// pour Gazebo, package:// pour le reel (URDF genere sur
la Jetson, affiche par RViz sur le ROG). IMU confirmee au lab (11,5 cm).

File: src/seekur_driver/urdf/seekur_jr_simple.urdf.xacro (robot description, xacro)
@@ -4,4 +4,17 @@
     <xacro:arg name="robot_color" default="Grey"/>
     <xacro:property name="robot_color" value="$(arg robot_color)"/>
+    <!-- Arguments specifiques au MATERIEL (2026-09-29).
+         Les valeurs par defaut sont celles de la SIMULATION : sim.launch.py
+         et les launch derives n'ont rien a passer. real.launch.py passe les
+         valeurs du vrai robot (meme logique que serial_port et linear_scale).
+           lidar_pitch_deg : inclinaison du LMS111 vers le haut. [SIM] 5 ;
+                             [LAB] 6.5 mesure (faisceau 40 cm a la sortie,
+                             52 cm a 1,05 m, 74 cm a 3 m).
+           mesh_uri        : prefixe des maillages. file:// + $(find) pour
+                             Gazebo ; package:// pour le reel, ou l'URDF est
+                             genere sur la Jetson et affiche par RViz sur le
+                             ROG (chemins absolus differents). -->
+    <xacro:arg name="lidar_pitch_deg" default="5"/>
+    <xacro:arg name="mesh_uri" default="file://$(find seekur_driver)/description/meshes"/>
     <!-- =======================================================
          Proprietes SeekurJR
@@ -43,5 +56,5 @@
          a la fois par RViz2 et par Gazebo Harmonic (package:// ne l'est
          pas toujours cote Gazebo). -->
-    <xacro:property name="mesh_dir" value="file://$(find seekur_driver)/description/meshes" />
+    <xacro:property name="mesh_dir" value="$(arg mesh_uri)" />
     <!-- Mat de camera. Le top du chassis est a (base_height - chassis_drop)
          dans base_link, soit 0.291 m ; la camera se deduit de la hauteur du
@@ -335,4 +348,6 @@
            acceleration centripete parasite en rotation lacet.
          z = -chassis_drop : le fond du chassis, soit 0.113 m du sol.
+           [LAB] 2026-09-29 : BNO055 fixe au centre, 11,5 cm du sol,
+           X vers l'avant, Z vers le haut -> modele juste a 2 mm pres.
            Plus bas que l'ancienne position a mi-hauteur, et donc plus
            proche du plan des axes de roue (z = 0) autour duquel se fait
@@ -361,5 +376,8 @@
              biaise les distances mur gauche / mur droit).
              A MESURER : distance centre du boitier <-> axe longitudinal. -->
-    <xacro:property name="lidar_pitch_deg" value="5" />      <!-- [SIM] inclinaison LiDAR vers le haut : evite le sol quand l avant replonge apres une bosse (a mesurer au lab) -->
+    <!-- Inclinaison vers le haut : argument lidar_pitch_deg (voir en tete).
+         [SIM] 5 : evite le sol quand l'avant replonge apres une bosse.
+         [LAB] 6.5 : mesure sur le vrai robot, passe par real.launch.py. -->
+    <xacro:property name="lidar_pitch_deg" value="$(arg lidar_pitch_deg)" />
     <joint name="laser_joint" type="fixed">
         <parent link="base_link" />

Commit message: Replace chassis mesh with seekurJr_moh

File: src/seekur_driver/urdf/seekur_jr_simple.urdf.xacro (robot description, xacro)
@@ -121,5 +121,5 @@
         <visual>
             <geometry>
-                <mesh filename="${mesh_dir}/seekurjr_chassis.obj" />
+                <mesh filename="${mesh_dir}/seekurJr_moh.obj" />
             </geometry>
             <origin xyz="0 0 0" rpy="0 0 0" />
