Commit message: urdf : train de roulement interchangeable (tripod | center)
- seekur_jr_simple.urdf.xacro : argument drivetrain (defaut tripod),
  macro drive_wheel commune, include drivetrain_<variante>.xacro.
- drivetrain_tripod.xacro : modele v10.2 deplace tel quel (URDF genere
  identique a main, verifie).
- drivetrain_center.xacro : roues motrices a x = 0 + roulettes avant et
  arriere sur joints prismatiques a ressort (springStiffness 3000 N/m,
  precharge 15 mm, amortissement 300 N.s/m). Joints de suspension
  publies dans /joint_states.
- sim.launch.py : argument drivetrain, herite par sim_ekf/sim_rtabmap/sim_yolo.
- MEMO.md : branche ajoutee aux travaux en cours.

Non teste dans Gazebo.

Co-Authored-By: Claude Opus 5.5 <noreply@anthropic.com>
Claude-Session: https://claude.ai/code/session_016jYge6uN3aJGjQF8BpsPjg

File: src/seekur_driver/urdf/seekur_jr_simple.urdf.xacro (robot description, xacro)
@@ -31,5 +31,5 @@
                           425 = empattement (axe avant - axe arriere)
                                 (utilise UNIQUEMENT pour placer les 4 roues
-                                visuelles ; la physique reste a 2 roues + roulette)
+                                visuelles ; la physique reste a 2 roues + roulette(s), voir drivetrain_*.xacro)
          ATTENTION - deux erreurs corrigees par rapport aux versions
          precedentes de ce fichier :
@@ -134,52 +134,49 @@
                           o_xyz="0 0 ${base_height / 2.0 - chassis_drop}" o_rpy="0 0 0" />
     </link>
-    <!-- Roue motrice right : PHYSIQUE SEULEMENT (collision + inertie).
+    <!-- ================================================================
+         TRAIN DE ROULEMENT INTERCHANGEABLE (2026-10-08)
+         Les 2 roues motrices PHYSIQUES (macro ci-dessous) sont communes ;
+         leur position, les roulettes et le JointStatePublisher Gazebo
+         viennent du fichier inclus, choisi par l'argument drivetrain :
+           tripod (defaut) : drivetrain_tripod.xacro
+                             roues a x = +base_length/4 + 1 roulette arriere
+                             (v10.2-tripode-traction-avant, valide sim et reel)
+           center          : drivetrain_center.xacro
+                             roues a x = 0 + 2 roulettes SUSPENDUES (ressort)
+                             avant/arriere : pivote au centre comme le vrai
+                             robot. NOUVEAU, a valider en sim.
+         Une valeur inconnue fait echouer xacro (fichier introuvable).
+         Le plugin DiffDrive (plus bas) est commun : memes noms de joints. -->
+    <xacro:arg name="drivetrain" default="tripod"/>
+    <!-- Roue motrice : PHYSIQUE SEULEMENT (collision + inertie).
          Pas de visuel : ce sont les 4 roues visuelles, aux positions
-         reelles, qui s'affichent (voir plus bas). -->
-    <link name="right_wheel_link">
-        <collision>
-            <geometry>
-                <cylinder radius="${wheel_radius}" length="${wheel_length}" />
-            </geometry>
-            <origin xyz="0 0 0" rpy="${pi / 2.0} 0 0" />
-        </collision>
-        <xacro:cylinder_inertia m="${wheel_mass}" r="${wheel_radius}" l="${wheel_length}"
-                               o_xyz="0 0 0" o_rpy="${pi / 2.0} 0 0" />
-    </link>
-    <!-- Roue motrice left : PHYSIQUE SEULEMENT (collision + inertie).
-         Pas de visuel : ce sont les 4 roues visuelles, aux positions
-         reelles, qui s'affichent (voir plus bas). -->
-    <link name="left_wheel_link">
-        <collision>
-            <geometry>
-                <cylinder radius="${wheel_radius}" length="${wheel_length}" />
-            </geometry>
-            <origin xyz="0 0 0" rpy="${pi / 2.0} 0 0" />
-        </collision>
-        <xacro:cylinder_inertia m="${wheel_mass}" r="${wheel_radius}" l="${wheel_length}"
-                               o_xyz="0 0 0" o_rpy="${pi / 2.0} 0 0" />
-    </link>
-    <!-- Roulette ARRIERE : PHYSIQUE SEULEMENT (absente du vrai SeekurJR,
-         gardee pour l'equilibre Gazebo du modele a 2 roues). Placee a
-         x = -base_length/3, elle est TIREE derriere le robot : elle roule
-         par-dessus les bosses au lieu d'y buter.
-         Touche le sol sans ecart (centre a -wheel_radius/2, rayon
-         wheel_radius/2) : trepied, pas de basculement.
-         Pas de visuel : elle apparaissait sous le chassis maille. -->
-    <link name="caster_wheel_link">
-        <collision>
-            <geometry>
-                <sphere radius="${wheel_radius / 2.0}" />
-            </geometry>
-            <origin xyz="0 0 0" rpy="0 0 0" />
-        </collision>
-        <xacro:sphere_inertia m="${caster_mass}" r="${wheel_radius / 2.0}"
-                             o_xyz="0 0 0" o_rpy="0 0 0" />
-    </link>
+         reelles, qui s'affichent (voir plus bas).
+         Y : depuis wheel_separation [DS] directement. NE PAS recalculer
+             depuis base_width + wheel_length : le chassis a un gap de
+             degagement avec le pneu, les deux grandeurs sont independantes. -->
+    <xacro:macro name="drive_wheel" params="side x y">
+        <link name="${side}_wheel_link">
+            <collision>
+                <geometry>
+                    <cylinder radius="${wheel_radius}" length="${wheel_length}" />
+                </geometry>
+                <origin xyz="0 0 0" rpy="${pi / 2.0} 0 0" />
+            </collision>
+            <xacro:cylinder_inertia m="${wheel_mass}" r="${wheel_radius}" l="${wheel_length}"
+                                   o_xyz="0 0 0" o_rpy="${pi / 2.0} 0 0" />
+        </link>
+        <joint name="base_${side}_wheel_joint" type="continuous">
+            <parent link="base_link" />
+            <child link="${side}_wheel_link" />
+            <origin xyz="${x} ${y} 0" rpy="0 0 0" />
+            <axis xyz="0 1 0" />
+        </joint>
+    </xacro:macro>
+    <xacro:include filename="drivetrain_$(arg drivetrain).xacro" />
     <!-- ================================================================
          Roues VISUELLES : les 4 roues du vrai SeekurJR, a leurs positions
          reelles (x = +/- wheelbase/2, y = +/- wheel_separation/2).
          - Aucune collision : la physique reste portee par les 2 roues
-           motrices avant + la roulette arriere.
+           motrices + la ou les roulettes (drivetrain_*.xacro).
          - Joint continuous avec <mimic> sur la roue motrice du meme cote :
            robot_state_publisher calcule leur angle a partir de
@@ -308,40 +305,4 @@
         <origin xyz="0 0 ${wheel_radius}" rpy="0 0 0"/>
     </joint>
-    <!-- Roues motrices.
-         Y : depuis wheel_separation [DS] directement. NE PAS recalculer
-             depuis base_width + wheel_length : le chassis a un gap de
-             degagement avec le pneu, les deux grandeurs sont independantes.
-         X : +base_length/4 (traction AVANT). Le vrai robot a 4 roues en
-             skid-steer ; ce modele en a 2 + une roulette arriere, donc
-             l'empattement reel (425 mm [DS]) ne s'applique pas ici.
-             Pourquoi l'avant : face a une bosse, les roues qui attaquent
-             l'obstacle doivent etre motrices ; une roulette poussee bute
-             et devient elle-meme l'obstacle. Valide sur mine_polycam.
-         Historique : v6-v9 = roues arriere + roulette avant ; v10.1 =
-         roues a x = 0 + 2 roulettes (gap 2 cm) : le chassis basculait
-         d'une roulette a l'autre (tangage +/-3.3 deg mesure a l'IMU sim)
-         et les fermetures de proximite RTAB-Map sont tombees de 5 a 0-1.
-         Abandonne.
-         LIMITE CONNUE - centre de rotation.
-         Le vrai SeekurJR pivote au milieu de son empattement (x = 0).
-         Ce modele pivote autour de l'axe de ses deux roues (x = +0.263),
-         donc en rotation pure l'arriere decrit un arc de 26 cm de rayon
-         au lieu de tourner sur place. Biais systematique, borne, connu.
-         Le LiDAR (x = 0.535) est plus proche du pivot qu'en traction
-         arriere, ce qui limite son deplacement en rotation.
-         Pour pivoter au centre sans basculer : roues a x = 0 + roulettes
-         SUSPENDUES (joint prismatique + ressort), pas un simple gap. -->
-    <joint name="base_right_wheel_joint" type="continuous">
-        <parent link="base_link" />
-        <child link="right_wheel_link" />
-        <origin xyz="${base_length / 4.0} ${-wheel_separation / 2.0} 0" rpy="0 0 0" />
-        <axis xyz="0 1 0" />
-    </joint>
-    <joint name="base_left_wheel_joint" type="continuous">
-        <parent link="base_link" />
-        <child link="left_wheel_link" />
-        <origin xyz="${base_length / 4.0} ${wheel_separation / 2.0} 0" rpy="0 0 0" />
-        <axis xyz="0 1 0" />
-    </joint>
     <!-- IMU monte au centre de la PLATEFORME BASSE du chassis.
          x = y = 0 : sur l'axe vertical de rotation du robot, donc aucune
@@ -358,9 +319,4 @@
         <child link="imu_link" />
         <origin xyz="0 0 ${-chassis_drop}" rpy="0 0 0" />
-    </joint>
-    <joint name="base_caster_wheel_joint" type="fixed">
-        <parent link="base_link" />
-        <child link="caster_wheel_link" />
-        <origin xyz="${-base_length / 3.0} 0 ${-wheel_radius / 2.0}" rpy="0 0 0" />
     </joint>
     <!-- LiDAR SICK, monte en saillie a l'AVANT sur support en equerre.
@@ -444,16 +400,4 @@
         </plugin>
     </gazebo>
-    <!-- ==================================================================
-         Plugin JointStatePublisher : UNE SEULE déclaration.
-         C'est lui qui produit l'état (position/vitesse) des roues côté
-         Gazebo. Ce flux doit ensuite être ponté vers ROS2 (/joint_states)
-         par ros_gz_bridge, sinon RViz2 affiche des roues figées.
-         ================================================================== -->
-    <gazebo>
-        <plugin filename="libgz-sim-joint-state-publisher-system.so" name="gz::sim::systems::JointStatePublisher">
-            <joint_name>base_left_wheel_joint</joint_name>
-            <joint_name>base_right_wheel_joint</joint_name>
-        </plugin>
-    </gazebo>
     <gazebo>
         <plugin filename="gz-sim-sensors-system" name="gz::sim::systems::Sensors">
@@ -595,9 +539,4 @@
     <!-- base_link et roues : plus de <material> Gazebo, les couleurs
          viennent des .mtl des maillages. -->
-    <gazebo reference="caster_wheel_link">
-        <material>Gazebo/Black</material>
-        <mu1 value="0.001" />
-        <mu2 value="0.001" />
-    </gazebo>
     <gazebo reference="laser_frame">
         <material>Gazebo/Grey</material>

Commit message: urdf : variante skid4 (4 roues motrices aux positions reelles)
drivetrain:=skid4 : 4 roues motrices a x = +/- wheelbase/2, aucune
roulette, comme le vrai SeekurJR (skid-steer). Frottement anisotrope
(longitudinal 1.0, lateral 0.6 via fdir1 = axe de roue).
Nouveau bloc extra_drive_joints dans le xacro principal : vide par
defaut (autres variantes inchangees), skid4 y ajoute ses 2 roues
arriere dans le plugin DiffDrive.
Limite : DiffDrive calcule l'odometrie en differentiel pur, donc
surestime la rotation en skid-steer ; l'EKF (IMU) corrige.

Co-Authored-By: Claude Opus 5.5 <noreply@anthropic.com>
Claude-Session: https://claude.ai/code/session_016jYge6uN3aJGjQF8BpsPjg

File: src/seekur_driver/urdf/seekur_jr_simple.urdf.xacro (robot description, xacro)
@@ -154,4 +154,8 @@
                              roues a x = 0 + roulette avant RIGIDE au sol
                              + roulette arriere SUSPENDUE (ressort).
+           skid4           : drivetrain_skid4.xacro
+                             4 roues motrices aux positions REELLES
+                             (x = +/-wheelbase/2), sans roulette : skid-steer
+                             comme le vrai SeekurJR.
          Une valeur inconnue fait echouer xacro (fichier introuvable).
          Le plugin DiffDrive (plus bas) est commun : memes noms de joints. -->
@@ -181,4 +185,8 @@
         </joint>
     </xacro:macro>
+    <!-- Roues motrices supplementaires a ajouter au plugin DiffDrive (plus
+         bas). Vide par defaut ; une variante a plus de 2 roues motrices
+         (skid4) redefinit ce bloc avec ses <left_joint>/<right_joint>. -->
+    <xacro:property name="extra_drive_joints"><!-- aucune roue motrice supplementaire --></xacro:property>
     <xacro:include filename="drivetrain_$(arg drivetrain).xacro" />
     <!-- ================================================================
@@ -389,4 +397,7 @@
             <right_joint>front_right_wheel_visual_joint</right_joint>
             <right_joint>rear_right_wheel_visual_joint</right_joint>
+            <!-- Roues motrices physiques supplementaires de la variante
+                 (vide sauf skid4, voir extra_drive_joints). -->
+            <xacro:insert_block name="extra_drive_joints" />
             <!-- Doivent rester coherents avec les proprietes xacro en tete
                  de fichier. Gazebo ne lit pas les ${} ici, d'ou la

Commit message: urdf : boite IMU remontee de 2 cm (ne depasse plus sous le chassis)
Le fond du maillage seekurJr_moh est a z = -0.081, 9 mm au-dessus du
fond mesure du chassis reel (-0.090) ou se trouve le repere imu_link.
Seul le visuel est decale ; le repere (TF, EKF, reel) reste a la
position mesuree au lab.

Co-Authored-By: Claude Opus 5.5 <noreply@anthropic.com>
Claude-Session: https://claude.ai/code/session_016jYge6uN3aJGjQF8BpsPjg

File: src/seekur_driver/urdf/seekur_jr_simple.urdf.xacro (robot description, xacro)
@@ -257,5 +257,10 @@
     <!-- IMU Link : monte sur la plateforme basse du chassis, sur l'axe
          vertical de rotation (voir imu_joint pour le detail du placement).
-         Petit box symbolique, inertie negligeable mais non nulle (exigence Gazebo). -->
+         Petit box symbolique, inertie negligeable mais non nulle (exigence Gazebo).
+         Visuel decale de +2 cm vers le haut (2026-10-08) : le fond du maillage
+         seekurJr_moh est a z = -0.081, 9 mm au-dessus du fond mesure du vrai
+         chassis (-0.090, ou est le repere imu_link). Sans decalage, la boite
+         rouge depassait sous le chassis. Le REPERE imu_link (TF, EKF) reste a
+         la position mesuree [LAB] ; seul le dessin bouge. -->
     <link name="imu_link">
         <visual>
@@ -263,5 +268,5 @@
                 <box size="0.03 0.03 0.02" />
             </geometry>
-            <origin xyz="0 0 0" rpy="0 0 0" />
+            <origin xyz="0 0 0.02" rpy="0 0 0" />
             <material name="red" />
         </visual>
