Commit message: urdf center : trim de precharge avant/arriere (assiette au repos)
Le CG est 8.7 mm en avant de l'axe (LiDAR + camera en porte-a-faux) :
en sim le robot piquait de ~0.6 deg au repos (avant +3.8 mm, arriere
-3.8 mm sur /joint_states). Precharge avant 18.2 mm, arriere 11.8 mm
(caster_trim = 3.2 mm) : meme charge totale sur les roulettes (90 N),
meme raideur en tangage, assiette au repos ramenee vers 0.

Co-Authored-By: Claude Opus 5.5 <noreply@anthropic.com>
Claude-Session: https://claude.ai/code/session_016jYge6uN3aJGjQF8BpsPjg

File: src/seekur_driver/urdf/drivetrain_center.xacro (robot description, xacro)
@@ -30,5 +30,6 @@
            q < 0   : roulette descendue (creux)
          Ressort : F = -k (q - q_ref), avec q_ref = -preload, donc au repos
-         sur sol plat (q = 0) chaque roulette appuie de k * preload.
+         sur sol plat (q = 0) chaque roulette appuie de k * preload
+         (preload = caster_preload +/- caster_trim, voir plus bas).
          Dimensionnement (robot ~78.5 kg, ~770 N) :
            k = 3000 N/m, preload 15 mm -> 45 N par roulette, soit ~12 % du
@@ -46,5 +47,13 @@
          Au-dela de travel, la roulette est en butee rigide comme en v10.1. -->
     <xacro:property name="caster_k" value="3000.0" />        <!-- N/m -->
-    <xacro:property name="caster_preload" value="0.015" />   <!-- m -->
+    <xacro:property name="caster_preload" value="0.015" />   <!-- m, moyenne avant/arriere -->
+    <!-- Correction d'assiette : le CG est 8.7 mm en avant de l'axe (LiDAR et
+         camera en porte-a-faux, couple ~6.7 N.m). Sans correction, le robot
+         pique du nez de ~0.5 deg (mesure sim 2026-10-08 : avant +3.8 mm,
+         arriere -3.8 mm). Precharge AVANT + trim, ARRIERE - trim :
+         6.7 N.m / 0.35 m / 2 roulettes = 9.6 N -> 9.6 / k = 3.2 mm.
+         Charge totale sur les roulettes inchangee (90 N). Seule l'assiette
+         au repos change ; la raideur en tangage reste la meme. -->
+    <xacro:property name="caster_trim" value="0.0032" />     <!-- m -->
     <xacro:property name="caster_damping" value="300.0" />   <!-- N.s/m -->
     <xacro:property name="caster_droop" value="0.03" />      <!-- m, descente max sous le sol plat -->
@@ -56,5 +65,5 @@
          Sphere quasi sans frottement sur joint prismatique vertical.
          Pas de visuel (masquee par le chassis maille). -->
-    <xacro:macro name="suspended_caster" params="name x">
+    <xacro:macro name="suspended_caster" params="name x preload">
         <link name="${name}_caster_link">
             <collision>
@@ -79,5 +88,5 @@
         <gazebo reference="base_${name}_caster_joint">
             <springStiffness>${caster_k}</springStiffness>
-            <springReference>${-caster_preload}</springReference>
+            <springReference>${-preload}</springReference>
         </gazebo>
         <gazebo reference="${name}_caster_link">
@@ -86,6 +95,6 @@
         </gazebo>
     </xacro:macro>
-    <xacro:suspended_caster name="front" x="${caster_x}" />
-    <xacro:suspended_caster name="rear"  x="${-caster_x}" />
+    <xacro:suspended_caster name="front" x="${caster_x}"  preload="${caster_preload + caster_trim}" />
+    <xacro:suspended_caster name="rear"  x="${-caster_x}" preload="${caster_preload - caster_trim}" />
     <!-- ==================================================================
          Plugin JointStatePublisher : UNE SEULE declaration (par variante).

Commit message: urdf : modele de reference seekur_jr.urdf.xacro (skid4), variantes a part
- seekur_jr.urdf.xacro (nouveau) : modele autonome sans include,
  skid-steer 4 roues motrices aux positions reelles, maillage porte par
  les roues physiques, chassis 44 kg (total 77.5 kg = datasheet),
  WheelSlip, capteurs identiques a la version precedente (verifie lien
  par lien). Charge par defaut par sim.launch.py (et sim_*, slam) et par
  real.launch.py (joint_state_publisher y publie les 4 roues : TF
  valides).
- seekur_jr_simple.urdf.xacro renomme seekur_jr_variants.urdf.xacro :
  variantes d'essai via drivetrain:=<nom> ; skid4 y passe aussi a 44 kg.
- sim.launch.py : drivetrain vide par defaut = modele de reference.
- README et MEMO a jour.

Co-Authored-By: Claude Opus 5.5 <noreply@anthropic.com>
Claude-Session: https://claude.ai/code/session_016jYge6uN3aJGjQF8BpsPjg

File: src/seekur_driver/urdf/drivetrain_center.xacro (robot description, xacro)
@@ -2,5 +2,5 @@
 <!-- =====================================================================
      Train de roulement CENTRE + 2 ROULETTES SUSPENDUES (drivetrain:=center)
-     Inclus par seekur_jr_simple.urdf.xacro, qui fournit les proprietes
+     Inclus par seekur_jr_variants.urdf.xacro, qui fournit les proprietes
      (base_length, wheel_radius, ...), les macros d'inertie et drive_wheel.
      NOUVEAU (2026-10-08), A VALIDER EN SIM. Reprend la geometrie de

File: src/seekur_driver/urdf/drivetrain_center_rear_spring.xacro (robot description, xacro)
@@ -3,5 +3,5 @@
      Train de roulement CENTRE + roulette AVANT RIGIDE + roulette ARRIERE
      SUSPENDUE (drivetrain:=center_rear_spring)
-     Inclus par seekur_jr_simple.urdf.xacro, qui fournit les proprietes
+     Inclus par seekur_jr_variants.urdf.xacro, qui fournit les proprietes
      (base_length, wheel_radius, ...), les macros d'inertie et drive_wheel.
      Compromis entre center (2 ressorts) et center_rigid (2 butees),

File: src/seekur_driver/urdf/drivetrain_center_rigid.xacro (robot description, xacro)
@@ -2,5 +2,5 @@
 <!-- =====================================================================
      Train de roulement CENTRE + 2 ROULETTES RIGIDES (drivetrain:=center_rigid)
-     Inclus par seekur_jr_simple.urdf.xacro, qui fournit les proprietes
+     Inclus par seekur_jr_variants.urdf.xacro, qui fournit les proprietes
      (base_length, wheel_radius, ...), les macros d'inertie et drive_wheel.
      Variante SANS RESSORT de drivetrain_center.xacro (2026-10-08) :

File: src/seekur_driver/urdf/drivetrain_skid4.xacro (robot description, xacro)
@@ -2,5 +2,5 @@
 <!-- =====================================================================
      Train de roulement SKID-STEER 4 ROUES (drivetrain:=skid4)
-     Inclus par seekur_jr_simple.urdf.xacro, qui fournit les proprietes
+     Inclus par seekur_jr_variants.urdf.xacro, qui fournit les proprietes
      (wheelbase, wheel_separation, ...), les macros d'inertie et drive_wheel.
      Copie de la cinematique du VRAI SeekurJR (2026-10-08) : 4 roues

File: src/seekur_driver/urdf/drivetrain_tripod.xacro (robot description, xacro)
@@ -2,5 +2,5 @@
 <!-- =====================================================================
      Train de roulement TRIPODE, traction AVANT (defaut, drivetrain:=tripod)
-     Inclus par seekur_jr_simple.urdf.xacro, qui fournit les proprietes
+     Inclus par seekur_jr_variants.urdf.xacro, qui fournit les proprietes
      (base_length, wheel_radius, ...), les macros d'inertie et drive_wheel.
      Geometrie identique a v10.2-tripode-traction-avant (2026-09-27).

File: src/seekur_driver/urdf/seekur_jr_variants.urdf.xacro (robot description, xacro)
@@ -17,4 +17,8 @@
     <xacro:arg name="lidar_pitch_deg" default="5"/>
     <xacro:arg name="mesh_uri" default="file://$(find seekur_driver)/description/meshes"/>
+    <!-- Train de roulement (voir drivetrain_*.xacro et le bloc TRAIN DE
+         ROULEMENT INTERCHANGEABLE plus bas). Ce fichier sert aux ESSAIS ; le
+         modele de reference est seekur_jr.urdf.xacro (skid4 seul). -->
+    <xacro:arg name="drivetrain" default="tripod"/>
     <!-- =======================================================
          Proprietes SeekurJR
@@ -69,5 +73,8 @@
            top chassis    = 0.113 + base_height       = 0.494 m du sol  [DS] OK -->
     <!-- Masses (datasheet : robot complet 77 kg) -->
-    <xacro:property name="base_mass" value="60.0" />         <!-- chassis + electronique -->
+    <!-- Chassis + electronique. Datasheet : robot complet 77 kg, roues
+         comprises. Variantes a 2 roues physiques : 60 + 2 x 8 + capteurs
+         ~1.5 = 77.5 kg. skid4 a 4 roues physiques : 44 + 4 x 8 + 1.5 = 77.5 kg. -->
+    <xacro:property name="base_mass" value="${44.0 if '$(arg drivetrain)' == 'skid4' else 60.0}" />
     <xacro:property name="wheel_mass" value="8.0" />         <!-- 16" pneumatique ~8 kg piece -->
     <xacro:property name="caster_mass" value="0.5" />        <!-- non present sur vrai SeekurJR, garde pour stabilite Gazebo -->
@@ -160,5 +167,5 @@
          Une valeur inconnue fait echouer xacro (fichier introuvable).
          Le plugin DiffDrive (plus bas) est commun : memes noms de joints. -->
-    <xacro:arg name="drivetrain" default="tripod"/>
+    <!-- (argument drivetrain declare en tete de fichier : base_mass en depend) -->
     <!-- Roue motrice : PHYSIQUE SEULEMENT (collision + inertie).
          Pas de visuel : ce sont les 4 roues visuelles, aux positions
